File: sketch/Counters/Counters.sch (KiCad schematic (older format))
At the start: 18 parts, among them U1 SN74ALS169BN, U10 SN74F163AN, U11 SN74F163AN, U12 SN74F163AN, U13 SN74AHCT573N, U14 SN74AHCT573N, U15 SN74AHCT573N, U16 SN74AHCT573N, U2 SN74ALS169BN, U3 SN74ALS169BN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

Commit message: counters
Parts:
- removed ADDRESS_BUS1, DATA_BUS1: Conn_01x16, Socket_Strips:Socket_Strip_Straight_1x16_Pitch2.54mm, symbol Connector_Generic:Conn_01x16
- removed U1, U2, U3, U4: SN74ALS169BN, Housings_DIP:DIP-16_W7.62mm, symbol additional_components:SN74ALS169BN
- removed U10, U11, U12, U9: SN74F163AN, Housings_DIP:DIP-16_W7.62mm, symbol additional_components:SN74F163AN
- removed U13, U14, U15, U16, U5, U6, U7, U8: SN74AHCT573N, Housings_DIP:DIP-20_W7.62mm, symbol additional_components:SN74AHCT573N
