File: sketch/Counters/Counters.kicad_pcb (KiCad board)
At the start: 2 copper layers, 19 parts, among them U1 SN74ALS169BN, U10 SN74F163AN, U11 SN74F163AN, U12 SN74F163AN, U13 SN74AHCT573N, U14 SN74AHCT573N, U15 SN74AHCT573N, U16 SN74AHCT573N, U2 SN74ALS169BN, U3 SN74ALS169BN, U4 SN74ALS169BN, U5 SN74AHCT573N, U6 SN74AHCT573N, U7 SN74AHCT573N, U8 SN74AHCT573N, U9 SN74F163AN

Commit message: counters
Parts:
- moved U3 135.4 mm to (186.7, 92.7)
- moved U1 135.3 mm to (166.4, 92.7)
- moved U2 126.7 mm to (166.4, 121.9)
- moved U4 117.7 mm to (186.7, 121.9)
- moved U8 92.7 mm to (148.6, 116.8)
- moved U5 66.2 mm to (148.6, 29.2)
- moved U7 58.2 mm to (148.6, 87.6)
- moved U6 54.0 mm to (148.6, 58.4)
- moved REF** 18.2 mm to (261.6, 25.4)
- moved ADDRESS_BUS1 16.6 mm to (227.3, 99.1)
- moved DATA_BUS1 14.0 mm to (227.3, 31.8)
- moved U10 8.89 mm to (166.4, 58.4)
- moved U9 8.89 mm to (166.4, 29.2)
- moved U11 8.89 mm to (186.7, 29.2)
- moved U12 8.89 mm to (186.7, 58.4)
Routing:
- net Net-(DATA_BUS1-Pad15): track 251.5 -> 48.4 mm
- net Net-(DATA_BUS1-Pad16): track 255.6 -> 52.6 mm
- net Net-(DATA_BUS1-Pad13): track 240.7 -> 52.6 mm
- net Net-(DATA_BUS1-Pad12): track 207.1 -> 38.4 mm
- net Net-(DATA_BUS1-Pad14): track 247.4 -> 82.0 mm
- net Net-(DATA_BUS1-Pad10): track 192.8 -> 30.1 mm
- net Net-(DATA_BUS1-Pad11): track 200.1 -> 39.6 mm
- net Net-(DATA_BUS1-Pad9): track 185.9 -> 30.1 mm
- net Net-(U10-Pad2): track 178.0 -> 45.2 mm
- net Net-(DATA_BUS1-Pad4): track 144.3 -> 26.5 mm
- net Net-(DATA_BUS1-Pad3): track 136.0 -> 26.5 mm
- net Net-(DATA_BUS1-Pad2): track 128.5 -> 26.5 mm
- net Net-(U10-Pad11): track 72.1 -> 0.00 mm
- net Net-(DATA_BUS1-Pad1): track 89.6 -> 26.5 mm
- net Net-(U10-Pad15): track 12.7 -> 65.3 mm
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
Commit message: counters
Parts:
- added J1: Conn_01x10, Connector_PinSocket_2.54mm:PinSocket_1x10_P2.54mm_Vertical, F.Cu at (168.9, 21.6)
Routing:
- net +5V: track 0.00 -> 563.0 mm
- net GND: track 0.00 -> 497.2 mm
- net /LDSP: track 0.00 -> 214.1 mm, vias 0 -> 1
- net /OEPCA: track 0.00 -> 157.0 mm, vias 0 -> 2
- net /OESPA: track 0.00 -> 130.9 mm
- net /LDPC: track 0.00 -> 102.4 mm, vias 0 -> 2
- net /DECSP: track 0.00 -> 95.9 mm, vias 0 -> 1
- net Net-(U10-Pad15): track 65.3 -> 0.00 mm
- net Net-(DATA_BUS1-Pad14): track 82.0 -> 18.9 mm
- net Net-(U13-Pad5): track 62.6 -> 0.00 mm
- net /OESPD: track 0.00 -> 60.7 mm
- net Net-(U10-Pad12): track 42.6 -> 0.00 mm
- net Net-(U10-Pad13): track 36.8 -> 0.00 mm
- net Net-(U10-Pad14): track 35.7 -> 0.00 mm
- net Net-(DATA_BUS1-Pad5): track 50.0 -> 15.2 mm
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
Commit message: registers
Parts:
- moved PC4 63.5 mm to (186.7, 121.9)
- moved SP2 63.5 mm to (166.4, 58.4)
- moved PC3 63.5 mm to (186.7, 92.7)
- moved SP1 63.5 mm to (166.4, 29.2)
- moved PC1 20.3 mm to (186.7, 29.2)
- moved PC2 20.3 mm to (186.7, 58.4)
- moved SP3 20.3 mm to (166.4, 92.7)
- moved SP4 20.3 mm to (166.4, 121.9)
- renumbered U9 to PC1, U10 to PC2, U11 to PC3, U12 to PC4, U15 to PCA, U16 to PCA, U13 to PCD, U14 to PCD, U1 to SP1, U2 to SP2, U3 to SP3, U4 to SP4, U7 to SPA, U8 to SPA, U5 to SPD, U6 to SPD
Routing:
- net +5V: track 563.0 -> 0.00 mm
- net GND: track 497.2 -> 0.00 mm
- net /LDSP: track 214.1 -> 0.00 mm, vias 1 -> 0
- net /OEPCA: track 157.0 -> 0.00 mm, vias 2 -> 0
- net /OESPA: track 130.9 -> 0.00 mm
- net /LDPC: track 102.4 -> 0.00 mm, vias 2 -> 0
- net /DECSP: track 95.9 -> 0.00 mm, vias 1 -> 0
- net /OESPD: track 60.7 -> 0.00 mm
- net Net-(DATA_BUS1-Pad7): track 51.0 -> 0.00 mm, vias 3 -> 0
- net Net-(U13-Pad4): track 50.5 -> 0.00 mm, vias 3 -> 0
- net Net-(U10-Pad2): track 41.8 -> 0.00 mm, vias 1 -> 0
- net Net-(U13-Pad3): track 39.1 -> 0.00 mm
- net Net-(U13-Pad2): track 32.6 -> 0.00 mm
- net Net-(DATA_BUS1-Pad4): track 26.5 -> 0.00 mm
- net Net-(DATA_BUS1-Pad2): track 26.5 -> 0.00 mm
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