File: sketch/PC/PC.sch (KiCad schematic (older format))
At the start: 10 parts

Commit message: registers
Parts:
- added J?: Conn_01x08, symbol Connector_Generic:Conn_01x08
- added U?: SN74AS1004AN, symbol additional_74:SN74AS1004AN
Connections:
- net +5V: now also U?.11 (LE), U?.11 (LE), U?.11 (LE), U?.11 (LE), U?.20 (Vcc), U?.20 (Vcc), U?.20 (Vcc), U?.20 (Vcc), J?.6 (Pin_6), U?.14 (Vcc)
- net GND: now also U?.10 (GND), U?.10 (GND), U?.10 (GND), U?.10 (GND), J?.7 (Pin_7), U?.7 (GND)
- net LD: now also U?.1 (1A)
- net at U?.11 (Qd): now also U?.5 (4D), U?.5 (4D) (x2)
- net at U?.12 (Qc): now also U?.4 (3D), U?.4 (3D) (x2)
- net at U?.13 (Qb): now also U?.3 (2D), U?.3 (2D) (x2)
- net at U?.14 (Qa): now also U?.2 (1D), U?.2 (1D) (x2)
- net INC: now reaches U?.2 (CLK)
- net INC: now also J?.2 (Pin_2)
- net at DATA_BUS.2 (Pin_2), U?.4 (B): now also U?.18 (2Q)
- net at DATA_BUS.3 (Pin_3), U?.5 (C): now also U?.17 (3Q)
- net at DATA_BUS.4 (Pin_4), U?.6 (D): now also U?.16 (4Q)
- net at U?.11 (Qd): now also U?.9 (8D), U?.9 (8D) (x2)
- net at U?.12 (Qc): now also U?.8 (7D), U?.8 (7D) (x2)
- net at U?.13 (Qb): now also U?.7 (6D), U?.7 (6D) (x2)
- net at U?.14 (Qa): now also U?.6 (5D), U?.6 (5D) (x2)
- net at DATA_BUS.5 (Pin_5), U?.3 (A): now also U?.15 (5Q)
- net at DATA_BUS.6 (Pin_6), U?.4 (B): now also U?.14 (6Q)
- net at DATA_BUS.7 (Pin_7), U?.5 (C): now also U?.13 (7Q)
- net at DATA_BUS.8 (Pin_8), U?.6 (D): now also U?.12 (8Q)
- net at DATA_BUS.9 (Pin_9), U?.3 (A): now also U?.19 (1Q)
- net at DATA_BUS.10 (Pin_10), U?.4 (B): now also U?.18 (2Q)
- net at DATA_BUS.11 (Pin_11), U?.5 (C): now also U?.17 (3Q)
- net at DATA_BUS.12 (Pin_12), U?.6 (D): now also U?.16 (4Q)
- net RCO: now reaches U?.15 (RCO)
- net RCO: now also J?.5 (Pin_5)
- net at DATA_BUS.13 (Pin_13), U?.3 (A): now also U?.15 (5Q)
- net at DATA_BUS.14 (Pin_14), U?.4 (B): now also U?.14 (6Q)
- net at DATA_BUS.15 (Pin_15), U?.5 (C): now also U?.13 (7Q)
- net at DATA_BUS.16 (Pin_16), U?.6 (D): now also U?.12 (8Q)
- net at ADDRESS_BUS.1 (Pin_1): now also U?.19 (1Q)
- net at ADDRESS_BUS.10 (Pin_10): now also U?.18 (2Q)
- net at ADDRESS_BUS.11 (Pin_11): now also U?.17 (3Q)
- net at ADDRESS_BUS.12 (Pin_12): now also U?.16 (4Q)
- net at ADDRESS_BUS.13 (Pin_13): now also U?.15 (5Q)
- net at ADDRESS_BUS.14 (Pin_14): now also U?.14 (6Q)
- net at ADDRESS_BUS.15 (Pin_15): now also U?.13 (7Q)
- net at ADDRESS_BUS.16 (Pin_16): now also U?.12 (8Q)
- net at ADDRESS_BUS.2 (Pin_2): now also U?.18 (2Q)
- net at ADDRESS_BUS.3 (Pin_3): now also U?.17 (3Q)
- net at ADDRESS_BUS.4 (Pin_4): now also U?.16 (4Q)
- net at ADDRESS_BUS.5 (Pin_5): now also U?.15 (5Q)
- net at ADDRESS_BUS.6 (Pin_6): now also U?.14 (6Q)
- net at ADDRESS_BUS.7 (Pin_7): now also U?.13 (7Q)
- net at ADDRESS_BUS.8 (Pin_8): now also U?.12 (8Q)
- net at ADDRESS_BUS.9 (Pin_9): now also U?.19 (1Q)
- net OED: now reaches U?.1 (OE)
- net OED: now also U?.1 (OE), U?.3 (2A)
- net OEA: now reaches U?.1 (OE)
- net OEA: now also U?.1 (OE), U?.5 (3A)
- new net: J?.1 (Pin_1), U?.2 (1Y)
- new net: J?.3 (Pin_3), U?.4 (2Y)
- new net: J?.4 (Pin_4), U?.6 (3Y)
Other:
- moved on the sheet: ADDRESS_BUS, DATA_BUS, U?
