File: sketch/Registers.kicad_pcb (KiCad board)
At the start: 2 copper layers, 12 parts, among them U1 SN74AHCT573N, U2 SN74AHCT573N, U3 SN74F574N, U4 SN74F574N, U5 SN74AHCT573N, U6 SN74AHCT573N, U7 SN74AHCT573N, U8 SN74AHCT573N, U9 SN74AS1004AN

Commit message: registers
Routing:
- net Net-(ADDRESS_BUS1-Pad2): track 0.00 -> 33.6 mm
- net Net-(ADDRESS_BUS1-Pad8): track 0.00 -> 33.6 mm
- net Net-(ADDRESS_BUS1-Pad7): track 0.00 -> 33.6 mm
- net Net-(ADDRESS_BUS1-Pad6): track 0.00 -> 33.6 mm
- net Net-(ADDRESS_BUS1-Pad4): track 0.00 -> 33.6 mm
- net Net-(ADDRESS_BUS1-Pad3): track 0.00 -> 33.6 mm
- net Net-(ADDRESS_BUS1-Pad1): track 0.00 -> 33.6 mm
- net Net-(ADDRESS_BUS1-Pad5): track 0.00 -> 33.6 mm
- net Net-(ADDRESS_BUS1-Pad16): track 0.00 -> 31.4 mm
- net Net-(ADDRESS_BUS1-Pad9): track 0.00 -> 31.4 mm
- net Net-(ADDRESS_BUS1-Pad15): track 0.00 -> 31.4 mm
- net Net-(ADDRESS_BUS1-Pad14): track 0.00 -> 31.4 mm
- net Net-(ADDRESS_BUS1-Pad13): track 0.00 -> 31.4 mm
- net Net-(ADDRESS_BUS1-Pad12): track 0.00 -> 31.4 mm
- net Net-(ADDRESS_BUS1-Pad11): track 0.00 -> 31.4 mm
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
Commit message: registers
Routing:
- net Net-(DATA_BUS1-Pad8): track 22.9 -> 186.7 mm
- net Net-(DATA_BUS1-Pad7): track 22.9 -> 179.8 mm
- net Net-(DATA_BUS1-Pad6): track 22.9 -> 172.9 mm
- net Net-(DATA_BUS1-Pad5): track 22.9 -> 165.7 mm
- net Net-(DATA_BUS1-Pad13): track 26.0 -> 167.5 mm
- net Net-(DATA_BUS1-Pad4): track 22.9 -> 158.7 mm
- net Net-(DATA_BUS1-Pad14): track 26.0 -> 160.5 mm
- net Net-(DATA_BUS1-Pad3): track 22.9 -> 151.8 mm
- net Net-(DATA_BUS1-Pad15): track 26.0 -> 153.6 mm
- net Net-(DATA_BUS1-Pad2): track 22.9 -> 144.8 mm
- net Net-(DATA_BUS1-Pad16): track 26.0 -> 142.8 mm
- net Net-(DATA_BUS1-Pad1): track 22.9 -> 111.7 mm
- net Net-(U3-Pad17): track 18.7 -> 77.7 mm
- net Net-(U3-Pad15): track 18.7 -> 77.7 mm
- net Net-(U3-Pad14): track 18.7 -> 77.7 mm
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